File: PCB/NeoGeo JAMMA OD.sch (EAGLE design)
At the start: 20 parts, among them U1A ESP32DEVKITC, U2A SN74AHCT125N, U3A SN74AHCT125N, U4A SN74AHCT125N

Commit message: ESP Size Change
The original design used an ESP with a 22mm spacing, Updated the part to the standard version with 25mm spacing.
Parts:
- removed U1A: ESP32DEVKITC, ESP32-DEVKITC:ESP32DEVKITC
- added U1: ESP32DEVKITC, ESP32-DEVKITC4:ESP32DEVKITC
Connections:
- net 3V3IN: now also U1.3V3, U1.SVN; no longer U1A.3V3, U1A.SVN
- net 5VIN: now also U1.5V; no longer U1A.5V
- net GND: now also U1.GND@38, U1.IO34, U1.IO35; no longer U1A.GND@38, U1A.IO34, U1A.IO35
- net IO17: now also U1.IO17; no longer U1A.IO17
- net IO18: now also U1.IO18; no longer U1A.IO18
- net IO19: now also U1.IO19; no longer U1A.IO19
- net IO21: now also U1.IO21; no longer U1A.IO21
- net IO22: now also U1.IO22; no longer U1A.IO22
- net IO23: now also U1.IO23; no longer U1A.IO23
- net IO25: now also U1.IO25; no longer U1A.IO25
- net IO26: now also U1.IO26; no longer U1A.IO26
- net IO27: now also U1.IO27; no longer U1A.IO27
- net IO3: now also U1.RXD0; no longer U1A.RXD0
- net IO32: now also U1.IO32; no longer U1A.IO32
- net IO33: now also U1.IO33; no longer U1A.IO33
- net IO5: now also U1.IO5; no longer U1A.IO5
Changed lines of the file:
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@@
 <part name="GND" library="wirepad" library_urn="urn:adsk.eagle:library:412" deviceset="SMD5" device="" package3d_urn="urn:adsk.eagle:package:30841/1"/>
 <part name="START" library="wirepad" library_urn="urn:adsk.eagle:library:412" deviceset="SMD5" device="" package3d_urn="urn:adsk.eagle:package:30841/1"/>
-<part name="U1A" library="ESP32-DEVKITC" deviceset="ESP32DEVKITC" device=""/>
 <part name="LED" library="adafruit" library_urn="urn:adsk.eagle:library:420" deviceset="LED" device="CHIPLED_1206" package3d_urn="urn:adsk.eagle:package:6240560/1"/>
 <part name="R3" library="adafruit" deviceset="R-US_" device="R1206" value="84"/>
@@
 <part name="A" library="wirepad" library_urn="urn:adsk.eagle:library:412" deviceset="SMD5" device="" package3d_urn="urn:adsk.eagle:package:30841/1"/>
 <part name="CREDIT" library="wirepad" library_urn="urn:adsk.eagle:library:412" deviceset="SMD5" device="" package3d_urn="urn:adsk.eagle:package:30841/1"/>
+<part name="U1" library="ESP32-DEVKITC4" deviceset="ESP32DEVKITC" device=""/>
 </parts>
 <sheets>
@@
 <attribute name="VALUE" x="349.377" y="-170.942" size="1.778" layer="96"/>
 </instance>
-<instance part="U1A" gate="G$1" x="218.44" y="-121.92" smashed="yes" rot="R270">
-<attribute name="NAME" x="223.52" y="-95.25" size="1.27" layer="95"/>
-</instance>
 <instance part="LED" gate="G$1" x="383.54" y="-154.94" smashed="yes">
 <attribute name="NAME" x="387.096" y="-159.512" size="1.778" layer="95" rot="R90"/>
@@
 <attribute name="NAME" x="339.217" y="-165.7858" size="1.778" layer="95"/>
 <attribute name="VALUE" x="349.377" y="-168.402" size="1.778" layer="96"/>
+</instance>
+<instance part="U1" gate="G$1" x="218.44" y="-121.92" smashed="yes" rot="R270">
+<attribute name="NAME" x="223.52" y="-95.25" size="1.27" layer="95"/>
 </instance>
 </instances>
@@
 </segment>
 <segment>
-<pinref part="U1A" gate="G$1" pin="GND@38"/>
 <wire x1="236.22" y1="-99.06" x2="238.76" y2="-99.06" width="0.1524" layer="91"/>
 <wire x1="238.76" y1="-99.06" x2="238.76" y2="-152.4" width="0.1524" layer="91"/>
 <pinref part="U$10" gate="G$1" pin="GND"/>
-<pinref part="U1A" gate="G$1" pin="IO35"/>
 <wire x1="238.76" y1="-152.4" x2="238.76" y2="-154.94" width="0.1524" layer="91"/>
 <wire x1="200.66" y1="-111.76" x2="198.12" y2="-111.76" width="0.1524" layer="91"/>
@@
 <wire x1="238.76" y1="-152.4" x2="198.12" y2="-152.4" width="0.1524" layer="91"/>
 <junction x="238.76" y="-152.4"/>
-<pinref part="U1A" gate="G$1" pin="IO34"/>
 <wire x1="200.66" y1="-109.22" x2="198.12" y2="-109.22" width="0.1524" layer="91"/>
 <wire x1="198.12" y1="-109.22" x2="198.12" y2="-111.76" width="0.1524" layer="91"/>
 <junction x="198.12" y="-111.76"/>
+<pinref part="U1" gate="G$1" pin="IO34"/>
+<pinref part="U1" gate="G$1" pin="IO35"/>
+<pinref part="U1" gate="G$1" pin="GND@38"/>
 </segment>
 </net>
@@
 </segment>
 <segment>
-<pinref part="U1A" gate="G$1" pin="5V"/>
 <wire x1="200.66" y1="-144.78" x2="193.04" y2="-144.78" width="0.1524" layer="91"/>
 <wire x1="193.04" y1="-144.78" x2="193.04" y2="-139.7" width="0.1524" layer="91"/>
 <pinref part="U$8" gate="G$1" pin="VIN"/>
 <label x="193.04" y="-144.78" size="1.778" layer="95" rot="R90"/>
+<pinref part="U1" gate="G$1" pin="5V"/>
 </segment>
 </net>
@@
 </segment>
 <segment>
-<pinref part="U1A" gate="G$1" pin="IO5"/>
 <wire x1="236.22" y1="-121.92" x2="248.92" y2="-121.92" width="0.1524" layer="91"/>
 <label x="243.84" y="-121.92" size="1.778" layer="95"/>
+<pinref part="U1" gate="G$1" pin="IO5"/>
 </segment>
 </net>
@@
 </segment>
 <segment>
-<pinref part="U1A" gate="G$1" pin="IO18"/>
 <wire x1="236.22" y1="-119.38" x2="248.92" y2="-119.38" width="0.1524" layer="91"/>
 <label x="243.84" y="-119.38" size="1.778" layer="95"/>
+<pinref part="U1" gate="G$1" pin="IO18"/>
 </segment>
 </net>
@@
 </segment>
 <segment>
-<pinref part="U1A" gate="G$1" pin="IO23"/>
 <wire x1="236.22" y1="-101.6" x2="248.92" y2="-101.6" width="0.1524" layer="91"/>
 <label x="243.84" y="-101.6" size="1.778" layer="95"/>
+<pinref part="U1" gate="G$1" pin="IO23"/>
 </segment>
 </net>
 <net name="IO26" class="0">
 <segment>
-<pinref part="U1A" gate="G$1" pin="IO26"/>
 <wire x1="200.66" y1="-121.92" x2="185.42" y2="-121.92" width="0.1524" layer="91"/>
 <label x="185.42" y="-121.92" size="1.778" layer="95"/>
+<pinref part="U1" gate="G$1" pin="IO26"/>
 </segment>
 <segment>
@@
 </segment>
 <segment>
-<pinref part="U1A" gate="G$1" pin="IO25"/>
 <wire x1="200.66" y1="-119.38" x2="185.42" y2="-119.38" width="0.1524" layer="91"/>
 <label x="185.42" y="-119.38" size="1.778" layer="95"/>
+<pinref part="U1" gate="G$1" pin="IO25"/>
 </segment>
 </net>
@@
 </segment>
 <segment>
-<pinref part="U1A" gate="G$1" pin="IO21"/>
 <wire x1="236.22" y1="-111.76" x2="248.92" y2="-111.76" width="0.1524" layer="91"/>
 <label x="243.84" y="-111.76" size="1.778" layer="95"/>
+<pinref part="U1" gate="G$1" pin="IO21"/>
 </segment>
 </net>
@@
 </segment>
 <segment>
-<pinref part="U1A" gate="G$1" pin="IO19"/>
 <wire x1="236.22" y1="-116.84" x2="248.92" y2="-116.84" width="0.1524" layer="91"/>
 <label x="243.84" y="-116.84" size="1.778" layer="95"/>
+<pinref part="U1" gate="G$1" pin="IO19"/>
 </segment>
 </net>
@@
 </segment>
 <segment>
-<pinref part="U1A" gate="G$1" pin="IO22"/>
 <wire x1="236.22" y1="-104.14" x2="248.92" y2="-104.14" width="0.1524" layer="91"/>
 <label x="243.84" y="-104.14" size="1.778" layer="95"/>
+<pinref part="U1" gate="G$1" pin="IO22"/>
 </segment>
 </net>
@@
 </segment>
 <segment>
-<pinref part="U1A" gate="G$1" pin="IO27"/>
 <wire x1="200.66" y1="-124.46" x2="185.42" y2="-124.46" width="0.1524" layer="91"/>
 <label x="185.42" y="-124.46" size="1.778" layer="95"/>
+<pinref part="U1" gate="G$1" pin="IO27"/>
 </segment>
 </net>
 <net name="IO33" class="0">
 <segment>
-<pinref part="U1A" gate="G$1" pin="IO33"/>
 <wire x1="200.66" y1="-116.84" x2="185.42" y2="-116.84" width="0.1524" layer="91"/>
 <label x="185.42" y="-116.84" size="1.778" layer="95"/>
+<pinref part="U1" gate="G$1" pin="IO33"/>
 </segment>
 <segment>
@@
 </segment>
 <segment>
-<pinref part="U1A" gate="G$1" pin="RXD0"/>
 <wire x1="248.92" y1="-109.22" x2="236.22" y2="-109.22" width="0.1524" layer="91"/>
 <label x="243.84" y="-109.22" size="1.778" layer="95"/>
+<pinref part="U1" gate="G$1" pin="RXD0"/>
 </segment>
 </net>
@@
 </segment>
 <segment>
-<pinref part="U1A" gate="G$1" pin="IO17"/>
 <wire x1="236.22" y1="-124.46" x2="248.92" y2="-124.46" width="0.1524" layer="91"/>
 <label x="243.84" y="-124.46" size="1.778" layer="95"/>
+<pinref part="U1" gate="G$1" pin="IO17"/>
 </segment>
 </net>
@@
 <net name="3V3IN" class="0">
 <segment>
-<pinref part="U1A" gate="G$1" pin="3V3"/>
 <wire x1="200.66" y1="-99.06" x2="198.12" y2="-99.06" width="0.1524" layer="91"/>
 <wire x1="198.12" y1="-99.06" x2="198.12" y2="-91.44" width="0.1524" layer="91"/>
 <pinref part="U$9" gate="G$1" pin="VIN"/>
-<pinref part="U1A" gate="G$1" pin="SVN"/>
 <wire x1="200.66" y1="-106.68" x2="198.12" y2="-106.68" width="0.1524" layer="91"/>
 <wire x1="198.12" y1="-106.68" x2="198.12" y2="-99.06" width="0.1524" layer="91"/>
 <junction x="198.12" y="-99.06"/>
 <label x="198.12" y="-106.68" size="1.778" layer="95" rot="R90"/>
+<pinref part="U1" gate="G$1" pin="3V3"/>
+<pinref part="U1" gate="G$1" pin="SVN"/>
 </segment>
 <segment>
@@
 <net name="IO32" class="0">
 <segment>
-<pinref part="U1A" gate="G$1" pin="IO32"/>
 <wire x1="200.66" y1="-114.3" x2="185.42" y2="-114.3" width="0.1524" layer="91"/>
 <label x="185.42" y="-114.3" size="1.778" layer="95"/>
-</segment>
-<segment>
+<pinref part="U1" gate="G$1" pin="IO32"/>
+</segment>
+<segment>
