File: PCB/Nintendo64.sch (EAGLE design)
At the start: 15 parts, among them U1 ESP32DEVKITC

Commit message: Updated PCBs
Parts:
- removed U1: ESP32DEVKITC, ESP32-DEVKITC:ESP32DEVKITC
- added U2: ESP32DEVKITC, ESP32-DEVKITC4:ESP32DEVKITC
Connections:
- net 3V3: now also U2.3V3, U2.SVN; no longer U1.3V3, U1.SVN
- net GND: now also U2.GND@14, U2.GND@32, U2.GND@38, U2.IO21, U2.IO22, U2.IO25, U2.IO32, U2.IO33, U2.IO34, U2.IO35; no longer U1.GND@14, U1.GND@32, U1.GND@38, U1.IO21, U1.IO22, U1.IO25, U1.IO32, U1.IO33, U1.IO34, U1.IO35
- net LED: now also U2.IO17; no longer U1.IO17
- net P1DATA: now also U2.IO19; no longer U1.IO19
- net P2DATA: now also U2.IO5; no longer U1.IO5
- net P3DATA: now also U2.IO26; no longer U1.IO26
- net P4DATA: now also U2.IO27; no longer U1.IO27
Changed lines of the file:
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@@
 </classes>
 <parts>
-<part name="U1" library="ESP32-DEVKITC" deviceset="ESP32DEVKITC" device=""/>
 <part name="U$2" library="Airquality_Sensor" library_urn="urn:adsk.eagle:library:16015176" deviceset="GND" device=""/>
 <part name="P1DATA" library="wirepad" library_urn="urn:adsk.eagle:library:412" deviceset="SMD5" device="" package3d_urn="urn:adsk.eagle:package:30841/1"/>
@@
 <part name="LED" library="adafruit" library_urn="urn:adsk.eagle:library:420" deviceset="LED" device="CHIPLED_1206" package3d_urn="urn:adsk.eagle:package:6240560/1"/>
 <part name="R1" library="adafruit" deviceset="R-US_" device="R1206" value="84"/>
+<part name="U2" library="ESP32-DEVKITC4" deviceset="ESP32DEVKITC" device=""/>
 </parts>
 <sheets>
@@
 </plain>
 <instances>
-<instance part="U1" gate="G$1" x="68.58" y="50.8" smashed="yes" rot="R270">
-<attribute name="NAME" x="73.66" y="77.47" size="1.27" layer="95"/>
-</instance>
 <instance part="U$2" gate="G$1" x="68.58" y="12.7" smashed="yes">
 <attribute name="VALUE" x="67.056" y="10.16" size="1.27" layer="96"/>
@@
 <attribute name="NAME" x="95.4786" y="74.93" size="1.778" layer="95" rot="R270"/>
 <attribute name="VALUE" x="90.678" y="74.93" size="1.778" layer="96" rot="R270"/>
+</instance>
+<instance part="U2" gate="G$1" x="68.58" y="50.8" smashed="yes" rot="R270">
+<attribute name="NAME" x="73.66" y="77.47" size="1.27" layer="95"/>
 </instance>
 </instances>
@@
 <pinref part="U$2" gate="G$1" pin="GND"/>
 <wire x1="68.58" y1="20.32" x2="68.58" y2="15.24" width="0.1524" layer="91"/>
-<pinref part="U1" gate="G$1" pin="GND@32"/>
 <wire x1="86.36" y1="58.42" x2="88.9" y2="58.42" width="0.1524" layer="91"/>
 <wire x1="48.26" y1="40.64" x2="48.26" y2="38.1" width="0.1524" layer="91"/>
@@
 <wire x1="48.26" y1="20.32" x2="68.58" y2="20.32" width="0.1524" layer="91"/>
 <junction x="68.58" y="20.32"/>
-<pinref part="U1" gate="G$1" pin="GND@14"/>
 <wire x1="50.8" y1="40.64" x2="48.26" y2="40.64" width="0.1524" layer="91"/>
 <junction x="48.26" y="40.64"/>
@@
 <wire x1="93.98" y1="35.56" x2="93.98" y2="33.02" width="0.1524" layer="91"/>
 <label x="81.28" y="20.32" size="1.778" layer="95"/>
-<pinref part="U1" gate="G$1" pin="GND@38"/>
 <wire x1="86.36" y1="73.66" x2="88.9" y2="73.66" width="0.1524" layer="91"/>
 <wire x1="88.9" y1="73.66" x2="88.9" y2="68.58" width="0.1524" layer="91"/>
 <junction x="88.9" y="58.42"/>
-<pinref part="U1" gate="G$1" pin="IO22"/>
 <wire x1="88.9" y1="68.58" x2="88.9" y2="60.96" width="0.1524" layer="91"/>
 <wire x1="88.9" y1="60.96" x2="88.9" y2="58.42" width="0.1524" layer="91"/>
 <wire x1="88.9" y1="68.58" x2="86.36" y2="68.58" width="0.1524" layer="91"/>
 <junction x="88.9" y="68.58"/>
-<pinref part="U1" gate="G$1" pin="IO35"/>
 <wire x1="50.8" y1="60.96" x2="48.26" y2="60.96" width="0.1524" layer="91"/>
 <wire x1="48.26" y1="60.96" x2="48.26" y2="58.42" width="0.1524" layer="91"/>
-<pinref part="U1" gate="G$1" pin="IO33"/>
 <wire x1="48.26" y1="58.42" x2="48.26" y2="55.88" width="0.1524" layer="91"/>
 <wire x1="48.26" y1="55.88" x2="48.26" y2="53.34" width="0.1524" layer="91"/>
@@
 <wire x1="50.8" y1="55.88" x2="48.26" y2="55.88" width="0.1524" layer="91"/>
 <junction x="48.26" y="55.88"/>
-<pinref part="U1" gate="G$1" pin="IO25"/>
 <wire x1="50.8" y1="53.34" x2="48.26" y2="53.34" width="0.1524" layer="91"/>
 <junction x="48.26" y="53.34"/>
-<pinref part="U1" gate="G$1" pin="IO32"/>
 <wire x1="50.8" y1="58.42" x2="48.26" y2="58.42" width="0.1524" layer="91"/>
 <junction x="48.26" y="58.42"/>
-<pinref part="U1" gate="G$1" pin="IO34"/>
 <wire x1="50.8" y1="63.5" x2="48.26" y2="63.5" width="0.1524" layer="91"/>
 <wire x1="48.26" y1="63.5" x2="48.26" y2="60.96" width="0.1524" layer="91"/>
 <junction x="48.26" y="60.96"/>
-<pinref part="U1" gate="G$1" pin="IO21"/>
 <wire x1="86.36" y1="60.96" x2="88.9" y2="60.96" width="0.1524" layer="91"/>
 <junction x="88.9" y="60.96"/>
+<pinref part="U2" gate="G$1" pin="IO34"/>
+<pinref part="U2" gate="G$1" pin="IO35"/>
+<pinref part="U2" gate="G$1" pin="IO32"/>
+<pinref part="U2" gate="G$1" pin="IO33"/>
+<pinref part="U2" gate="G$1" pin="IO25"/>
+<pinref part="U2" gate="G$1" pin="GND@14"/>
+<pinref part="U2" gate="G$1" pin="GND@32"/>
+<pinref part="U2" gate="G$1" pin="IO21"/>
+<pinref part="U2" gate="G$1" pin="IO22"/>
+<pinref part="U2" gate="G$1" pin="GND@38"/>
 </segment>
 </net>
 <net name="P3DATA" class="0">
 <segment>
-<pinref part="U1" gate="G$1" pin="IO26"/>
 <pinref part="P3DATA" gate="1" pin="P"/>
 <wire x1="50.8" y1="50.8" x2="43.18" y2="50.8" width="0.1524" layer="91"/>
+<pinref part="U2" gate="G$1" pin="IO26"/>
 </segment>
 </net>
 <net name="P1DATA" class="0">
 <segment>
-<pinref part="U1" gate="G$1" pin="IO19"/>
 <pinref part="P1DATA" gate="1" pin="P"/>
 <wire x1="86.36" y1="55.88" x2="104.14" y2="55.88" width="0.1524" layer="91"/>
+<pinref part="U2" gate="G$1" pin="IO19"/>
 </segment>
 </net>
 <net name="P2DATA" class="0">
 <segment>
-<pinref part="U1" gate="G$1" pin="IO5"/>
 <pinref part="P2DATA" gate="1" pin="P"/>
 <wire x1="86.36" y1="50.8" x2="104.14" y2="50.8" width="0.1524" layer="91"/>
+<pinref part="U2" gate="G$1" pin="IO5"/>
 </segment>
 </net>
 <net name="P4DATA" class="0">
 <segment>
-<pinref part="U1" gate="G$1" pin="IO27"/>
 <wire x1="50.8" y1="48.26" x2="43.18" y2="48.26" width="0.1524" layer="91"/>
 <pinref part="P4DATA" gate="1" pin="P"/>
+<pinref part="U2" gate="G$1" pin="IO27"/>
 </segment>
 </net>
@@
 <wire x1="93.98" y1="48.26" x2="93.98" y2="43.18" width="0.1524" layer="91"/>
 <junction x="93.98" y="48.26"/>
-<pinref part="U1" gate="G$1" pin="IO17"/>
 <wire x1="86.36" y1="48.26" x2="93.98" y2="48.26" width="0.1524" layer="91"/>
 <junction x="93.98" y="48.26"/>
 <label x="93.98" y="58.42" size="1.778" layer="95" rot="R90"/>
+<pinref part="U2" gate="G$1" pin="IO17"/>
 </segment>
 </net>
@@
 <wire x1="43.18" y1="71.12" x2="45.72" y2="71.12" width="0.1524" layer="91"/>
 <junction x="45.72" y="71.12"/>
-<pinref part="U1" gate="G$1" pin="3V3"/>
 <wire x1="50.8" y1="73.66" x2="48.26" y2="73.66" width="0.1524" layer="91"/>
 <wire x1="48.26" y1="73.66" x2="48.26" y2="81.28" width="0.1524" layer="91"/>
@@
 <wire x1="93.98" y1="81.28" x2="93.98" y2="76.2" width="0.1524" layer="91"/>
 <label x="68.58" y="81.28" size="1.778" layer="95"/>
-<pinref part="U1" gate="G$1" pin="SVN"/>
 <wire x1="50.8" y1="66.04" x2="48.26" y2="66.04" width="0.1524" layer="91"/>
 <wire x1="48.26" y1="66.04" x2="48.26" y2="73.66" width="0.1524" layer="91"/>
@@
 <junction x="45.72" y="66.04"/>
 <junction x="48.26" y="66.04"/>
-</segment>
-</net>
+<pinref part="U2" gate="G$1" pin="3V3"/>
+<pinref part="U2" gate="G$1" pin="SVN"/>
+</segment>
+</net>
