File: PCB/PSX-PS2.brd (EAGLE design)
At the start: 73 x 29 mm, 19 parts, among them U1 ESP32DEVKITC

Commit message: Updated PCBs
Parts:
- U1: device ESP32-DEVKITC:ESP32-DEVKITC -> ESP32-DEVKITC4:ESP32-DEVKITC
- moved LED 1.00 mm to (25.2, 23.9)
- moved P2-1 1.00 mm to (36.0, 22.0)
- moved P2-2 1.00 mm to (41.0, 22.0)
- moved P2-3 1.00 mm to (46.0, 22.0)
- moved P2-4 1.00 mm to (51.0, 22.0)
- moved U1 0.87 mm to (31.2, 15.0)
Routing:
- net 3V3: track 103.6 -> 110.5 mm
- net P2-7: track 31.5 -> 34.7 mm
- net 8V: track 30.5 -> 33.5 mm
- net P1-6: track 54.1 -> 57.1 mm
- net P2-9: track 35.9 -> 38.1 mm
- net P1-2: track 44.0 -> 45.8 mm
- net P2-2: track 8.73 -> 10.4 mm
- net P2-1: track 37.3 -> 39.0 mm
- net LED: track 34.7 -> 36.0 mm
- net P1-7: track 52.6 -> 53.9 mm
- net P1-1: track 55.2 -> 56.1 mm
- net P2-6: track 16.3 -> 17.0 mm
- net P1-9: track 47.6 -> 48.3 mm
Other:
- board size 73 x 29 mm -> 73 x 31 mm
- board text added: "PSX/PS2 v2.0 9/13/23"
- board text removed: "PSX/PS2 v1.0 5/2/22"
