File: PCB/PSX-PS2.sch (EAGLE design)
At the start: 19 parts, among them U1 ESP32DEVKITC

Commit message: Updated PCBs
Parts:
- U1: device ESP32-DEVKITC:ESP32DEVKITC -> ESP32-DEVKITC4:ESP32DEVKITC
Changed lines of the file:
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@@
 </classes>
 <parts>
-<part name="U1" library="ESP32-DEVKITC" deviceset="ESP32DEVKITC" device=""/>
 <part name="U$2" library="Airquality_Sensor" library_urn="urn:adsk.eagle:library:16015176" deviceset="GND" device=""/>
 <part name="P1-1" library="wirepad" library_urn="urn:adsk.eagle:library:412" deviceset="SMD5" device="" package3d_urn="urn:adsk.eagle:package:30841/1"/>
@@
 <part name="P1-4" library="wirepad" library_urn="urn:adsk.eagle:library:412" deviceset="SMD5" device="" package3d_urn="urn:adsk.eagle:package:30841/1"/>
 <part name="P2-4" library="wirepad" library_urn="urn:adsk.eagle:library:412" deviceset="SMD5" device="" package3d_urn="urn:adsk.eagle:package:30841/1"/>
+<part name="U1" library="ESP32-DEVKITC4" deviceset="ESP32DEVKITC" device=""/>
 </parts>
 <sheets>
@@
 </plain>
 <instances>
-<instance part="U1" gate="G$1" x="68.58" y="50.8" smashed="yes" rot="R270">
-<attribute name="NAME" x="73.66" y="77.47" size="1.27" layer="95"/>
-</instance>
 <instance part="U$2" gate="G$1" x="68.58" y="15.24" smashed="yes">
 <attribute name="VALUE" x="67.056" y="12.7" size="1.27" layer="96"/>
@@
 <attribute name="NAME" x="31.877" y="37.4142" size="1.778" layer="95"/>
 <attribute name="VALUE" x="39.497" y="34.798" size="1.778" layer="96"/>
+</instance>
+<instance part="U1" gate="G$1" x="68.58" y="50.8" smashed="yes" rot="R270">
+<attribute name="NAME" x="73.66" y="77.47" size="1.27" layer="95"/>
 </instance>
 </instances>
@@
 <pinref part="U$2" gate="G$1" pin="GND"/>
 <wire x1="68.58" y1="20.32" x2="68.58" y2="17.78" width="0.1524" layer="91"/>
-<pinref part="U1" gate="G$1" pin="GND@32"/>
 <wire x1="86.36" y1="58.42" x2="88.9" y2="58.42" width="0.1524" layer="91"/>
 <junction x="88.9" y="58.42"/>
-<pinref part="U1" gate="G$1" pin="GND@38"/>
 <wire x1="86.36" y1="73.66" x2="88.9" y2="73.66" width="0.1524" layer="91"/>
 <wire x1="88.9" y1="73.66" x2="88.9" y2="58.42" width="0.1524" layer="91"/>
@@
 <wire x1="48.26" y1="20.32" x2="68.58" y2="20.32" width="0.1524" layer="91"/>
 <junction x="68.58" y="20.32"/>
-<pinref part="U1" gate="G$1" pin="GND@14"/>
 <wire x1="50.8" y1="40.64" x2="48.26" y2="40.64" width="0.1524" layer="91"/>
 <wire x1="93.98" y1="33.02" x2="88.9" y2="33.02" width="0.1524" layer="91"/>
@@
 <wire x1="43.18" y1="38.1" x2="48.26" y2="38.1" width="0.1524" layer="91"/>
 <junction x="48.26" y="38.1"/>
-<pinref part="U1" gate="G$1" pin="SVN"/>
 <wire x1="50.8" y1="66.04" x2="48.26" y2="66.04" width="0.1524" layer="91"/>
 <wire x1="48.26" y1="66.04" x2="48.26" y2="60.96" width="0.1524" layer="91"/>
-<pinref part="U1" gate="G$1" pin="IO35"/>
 <wire x1="48.26" y1="60.96" x2="48.26" y2="40.64" width="0.1524" layer="91"/>
 <wire x1="50.8" y1="60.96" x2="48.26" y2="60.96" width="0.1524" layer="91"/>
 <junction x="48.26" y="60.96"/>
+<pinref part="U1" gate="G$1" pin="SVN"/>
+<pinref part="U1" gate="G$1" pin="IO35"/>
+<pinref part="U1" gate="G$1" pin="GND@14"/>
+<pinref part="U1" gate="G$1" pin="GND@32"/>
+<pinref part="U1" gate="G$1" pin="GND@38"/>
 </segment>
 </net>
 <net name="3V3" class="0">
 <segment>
-<pinref part="U1" gate="G$1" pin="3V3"/>
 <wire x1="50.8" y1="73.66" x2="48.26" y2="73.66" width="0.1524" layer="91"/>
 <wire x1="48.26" y1="73.66" x2="48.26" y2="81.28" width="0.1524" layer="91"/>
@@
 <pinref part="R1" gate="G$1" pin="1"/>
 <wire x1="48.26" y1="81.28" x2="60.96" y2="81.28" width="0.1524" layer="91"/>
+<pinref part="U1" gate="G$1" pin="3V3"/>
 </segment>
 </net>
@@
 <pinref part="LED" gate="G$1" pin="A"/>
 <wire x1="93.98" y1="48.26" x2="93.98" y2="43.18" width="0.1524" layer="91"/>
-<pinref part="U1" gate="G$1" pin="IO17"/>
 <wire x1="86.36" y1="48.26" x2="93.98" y2="48.26" width="0.1524" layer="91"/>
 <label x="78.74" y="81.28" size="1.778" layer="95"/>
@@
 <wire x1="93.98" y1="81.28" x2="93.98" y2="48.26" width="0.1524" layer="91"/>
 <junction x="93.98" y="48.26"/>
+<pinref part="U1" gate="G$1" pin="IO17"/>
 </segment>
 </net>
 <net name="P2-7" class="0">
 <segment>
-<pinref part="U1" gate="G$1" pin="IO26"/>
 <pinref part="P2-7" gate="1" pin="P"/>
 <wire x1="50.8" y1="50.8" x2="43.18" y2="50.8" width="0.1524" layer="91"/>
+<pinref part="U1" gate="G$1" pin="IO26"/>
 </segment>
 </net>
 <net name="P1-7" class="0">
 <segment>
-<pinref part="U1" gate="G$1" pin="IO33"/>
 <wire x1="50.8" y1="55.88" x2="43.18" y2="55.88" width="0.1524" layer="91"/>
 <pinref part="P1-7" gate="1" pin="P"/>
+<pinref part="U1" gate="G$1" pin="IO33"/>
 </segment>
 </net>
 <net name="P2-6" class="0">
 <segment>
-<pinref part="U1" gate="G$1" pin="IO5"/>
 <pinref part="P2-6" gate="1" pin="P"/>
 <wire x1="86.36" y1="50.8" x2="96.52" y2="50.8" width="0.1524" layer="91"/>
+<pinref part="U1" gate="G$1" pin="IO5"/>
 </segment>
 </net>
 <net name="P1-1" class="0">
 <segment>
-<pinref part="U1" gate="G$1" pin="IO19"/>
 <pinref part="P1-1" gate="1" pin="P"/>
 <wire x1="86.36" y1="55.88" x2="96.52" y2="55.88" width="0.1524" layer="91"/>
+<pinref part="U1" gate="G$1" pin="IO19"/>
 </segment>
 </net>
 <net name="P1-9" class="0">
 <segment>
-<pinref part="U1" gate="G$1" pin="IO21"/>
 <wire x1="86.36" y1="60.96" x2="96.52" y2="60.96" width="0.1524" layer="91"/>
 <pinref part="P1-9" gate="1" pin="P"/>
+<pinref part="U1" gate="G$1" pin="IO21"/>
 </segment>
 </net>
 <net name="P2-1" class="0">
 <segment>
-<pinref part="U1" gate="G$1" pin="IO22"/>
 <wire x1="86.36" y1="68.58" x2="96.52" y2="68.58" width="0.1524" layer="91"/>
 <pinref part="P2-1" gate="1" pin="P"/>
+<pinref part="U1" gate="G$1" pin="IO22"/>
 </segment>
 </net>
 <net name="P2-2" class="0">
 <segment>
-<pinref part="U1" gate="G$1" pin="IO27"/>
 <pinref part="P2-2" gate="1" pin="P"/>
 <wire x1="50.8" y1="48.26" x2="43.18" y2="48.26" width="0.1524" layer="91"/>
+<pinref part="U1" gate="G$1" pin="IO27"/>
 </segment>
 </net>
 <net name="P2-9" class="0">
 <segment>
-<pinref part="U1" gate="G$1" pin="IO25"/>
 <wire x1="50.8" y1="53.34" x2="43.18" y2="53.34" width="0.1524" layer="91"/>
 <pinref part="P2-9" gate="1" pin="P"/>
+<pinref part="U1" gate="G$1" pin="IO25"/>
 </segment>
 </net>
 <net name="P1-2" class="0">
 <segment>
-<pinref part="U1" gate="G$1" pin="IO32"/>
 <wire x1="50.8" y1="58.42" x2="43.18" y2="58.42" width="0.1524" layer="91"/>
 <pinref part="P1-2" gate="1" pin="P"/>
+<pinref part="U1" gate="G$1" pin="IO32"/>
 </segment>
 </net>
 <net name="P1-6" class="0">
 <segment>
-<pinref part="U1" gate="G$1" pin="IO34"/>
 <wire x1="50.8" y1="63.5" x2="43.18" y2="63.5" width="0.1524" layer="91"/>
 <pinref part="P1-6" gate="1" pin="P"/>
+<pinref part="U1" gate="G$1" pin="IO34"/>
 </segment>
 </net>
 <net name="8V" class="0">
 <segment>
-<pinref part="U1" gate="G$1" pin="5V"/>
 <pinref part="P1-3" gate="1" pin="P"/>
 <wire x1="50.8" y1="27.94" x2="45.72" y2="27.94" width="0.1524" layer="91"/>
@@
 <wire x1="45.72" y1="25.4" x2="45.72" y2="27.94" width="0.1524" layer="91"/>
 <junction x="45.72" y="27.94"/>
-</segment>
-</net>
+<pinref part="U1" gate="G$1" pin="5V"/>
+</segment>
+</net>
